Commit message: robot frame tested in Rviz

File: src/robocap_sim/urdf/robot_core.xacro (robot description, xacro)
@@ -16,5 +16,5 @@
         <visual>
             <geometry>
-                <mesh filename="package://rbc_base/meshes/frame_ultra_low_poly.stl" scale="0.001 0.001 0.001"/>
+                <mesh filename="package://robocap_sim/urdf/frame_ultra_low_poly.stl" scale="0.001 0.001 0.001"/>
             </geometry>
             <material name="white"/>

Commit message: robot can be spawned in gazebo
But without the chassis mesh atm

File: src/robocap_sim/urdf/robot_core.xacro (robot description, xacro)
@@ -15,6 +15,9 @@
     <link name="chassis">
         <visual>
+            <origin xyz="0 0 0.75" rpy="0 0 0"/>
             <geometry>
-                <mesh filename="package://robocap_sim/urdf/frame_ultra_low_poly.stl" scale="0.001 0.001 0.001"/>
+                <!-- <mesh filename="package://robocap_sim/urdf/frame_ultra_low_poly.stl" scale="0.001 0.001 0.001"/> -->
+                        <!-- Offset the origin by half the height -->
+                    <box size="0.54 0.54 1.5"/>
             </geometry>
             <material name="white"/>
@@ -176,7 +179,7 @@
         </actuator>
     </transmission>
-    <gazebo>
+    <!-- <gazebo>
         <plugin name="gazebo_ros2_control" filename="libgazebo_ros2_control.so">
         </plugin>
-    </gazebo>
+    </gazebo> -->
 </robot>

Commit message: works in gazebo

File: src/robocap_sim/urdf/robot_core.xacro (robot description, xacro)
@@ -12,12 +12,12 @@
         <origin xyz="0 0 0"/>
     </joint>
-    <!-- chassis description goes here. It describes the chassis of the bot which is a 54cm x 54cm x 150cm box -->
+    <!-- chassis description goes here -->
     <link name="chassis">
         <visual>
-            <origin xyz="0 0 0.75" rpy="0 0 0"/>
             <geometry>
+                <!-- This works in Rviz -->
                 <!-- <mesh filename="package://robocap_sim/urdf/frame_ultra_low_poly.stl" scale="0.001 0.001 0.001"/> -->
-                        <!-- Offset the origin by half the height -->
-                    <box size="0.54 0.54 1.5"/>
+                <!-- This works in gazebo -->
+                <mesh filename="$(find robocap_sim)/urdf/frame_ultra_low_poly.stl" scale="0.001 0.001 0.001"/>
             </geometry>
             <material name="white"/>
@@ -179,7 +179,7 @@
         </actuator>
     </transmission>
-    <!-- <gazebo>
+    <gazebo>
         <plugin name="gazebo_ros2_control" filename="libgazebo_ros2_control.so">
         </plugin>
-    </gazebo> -->
+    </gazebo>
 </robot>
